Commit message: testing move base

File: robo_bringup/urdf/skidsteerV1.urdf (robot description, URDF)
Before this commit: robot skidsteerV1, 7 links, 6 joints
Links:
- removed link cam_f_l_link
- removed link cam_f_r_link
- added link cam_left_link
- added link cam_right_link
- added link odom_front
Joints:
- removed joint cam_f_l_joint
- removed joint cam_f_r_joint
- removed joint lidar_f_l_joint
- removed joint lidar_f_r_joint
- added joint cam_left_joint: type fixed, parent base_link, child cam_left_link, origin xyz=1 0.6 2.2 rpy=-1.57 0 -1.57
- added joint cam_right_joint: type fixed, parent base_link, child cam_right_link, origin xyz=1 -0.6 2.2 rpy=-1.57 0 -1.57
- added joint livox_left_joint: type fixed, parent base_link, child livox_left_frame, origin xyz=1 0.6 2.0 rpy=0 0 0
- added joint livox_right_joint: type fixed, parent base_link, child livox_right_frame, origin xyz=1 -0.6 2.0 rpy=0 0 0

Commit message: Auto stash before merge of "main" and "origin/main"
add sequence record

File: robo_bringup/urdf/skidsteerV1.urdf (robot description, URDF)
Before this commit: robot skidsteerV1, 8 links, 6 joints
Links:
- removed link odom_front
Joints:
- joint livox_left_joint: origin xyz=1 0.6 2.0 rpy=0 0 0 -> xyz=1 0.6 2.0 rpy=-3.1416 0 0
- joint livox_right_joint: origin xyz=1 -0.6 2.0 rpy=0 0 0 -> xyz=1 -0.6 2.0 rpy=-3.1416 0 0
